Commit message: add dynamic table generator, config, and update simulation spawn documentation

File: ros/steve_sim_prep/models/table/table.urdf (robot description, URDF)
Before this commit: robot inspection_table, 1 links, 0 joints
Links:
- link table_link: geometry collision box size=0.6 0.9 0.4; visual box size=0.6 0.9 0.4
