Commit message: Restore CAD NBV pipeline and add cuRobo start pose
- main.py: CAD-only pipeline (no SAM2, no supervisor/worker) in 5 stages:
  start pose -> CAD & surface sampling -> viewpoints & IK -> NBV loop -> export
- Start pose: camera position + look-at point in robot base frame
  (config defaults, --start-pos / --look-at), planned with cuRobo and verified
- Fix CAD mesh placement: apply URDF inertial offset (was 18-100 mm off)
- Capture from the measured camera pose; hide D435 housing during render
  (TinyRenderer stalled for minutes rendering from inside it)
- Coverage back to 8 mm threshold with normal consistency check
- Rerun viz restored (3D Inspection + Pipeline Benchmark Tree), shows start pose image

Co-Authored-By: Claude Opus 5 <noreply@anthropic.com>

File: sim/models/steve.urdf (robot description, URDF)
Before this commit: robot steve, 37 links, 36 joints
Joints:
- joint dummy_camera_joint: origin xyz=0.02 0.0 -0.06 rpy=1.57 3.14 1.57 -> xyz=0.0824968606369 0.0375010071413 -0.0928999999396 rpy=3.14159265358 2.05103933837e-10 -3.14158895358
